Commit message: wip

File: robotis_mini_model/urdf/leg.urdf.xacro (robot description, xacro)
@@ -2,8 +2,19 @@
 <robot xmlns:xacro="http://www.ros.org/wiki/xacro" name="robotis_mini">
   <xacro:include filename="$(find robotis_mini_model)/urdf/components.urdf.xacro"/>
-  <xacro:macro name="leg" params="name parent_link origin_xyz origin_rpy">
-    <xacro:robotis_mini_link name="${name}_upper_link" xyz="${origin_xyz}" rpy="${origin_rpy}" mesh_file="DMF-B01(W).stl"/>
-    <xacro:robotis_mini_link name="${name}_lower_link" xyz="0 0 0" rpy="0 0 0" mesh_file="DMF-B01(W).stl"/>
-    <xacro:robotis_mini_link name="${name}_foot_link" xyz="0 0 0" rpy="0 0 0" mesh_file="DMF-B01(W).stl"/>
+  <xacro:macro name="leg" params="name parent_link origin_xyz origin_rpy mirror">
+    <xacro:robotis_mini_link name="${name}_m1_plate" origin_xyz="${origin_xyz}" origin_rpy="${origin_rpy}" mesh_file="SPD-3B5(W).stl"/>
+    <xacro:robotis_mini_revolute_joint name="${parent_link}_to_${name}_m1_plate" parent_link="${parent_link}" child_link="${name}_m1_plate" axis_xyz="0 1 0" origin_xyz="0 0.1 0" origin_rpy="0 0 0" />
+    <xacro:robotis_mini_motor name="${name}_m1" origin_xyz="0 0 0" origin_rpy="0 0 0"/>
+    <xacro:robotis_mini_fixed_joint name="${name}_m1_plate_to_${name}_m1" parent_link="${name}_m1_plate" child_link="${name}_m1" origin_xyz="0.012 0.013 0" origin_rpy="${PI} ${PI} ${-PI/2.0}" />
+    <xacro:robotis_mini_link name="${name}_m1_plate2" origin_xyz="0 0 0" origin_rpy="0 0 0" mesh_file="SPU-5(W).stl"/>
+    <xacro:robotis_mini_fixed_joint name="${name}_m1_to_${name}_m1_plate2" parent_link="${name}_m1" child_link="${name}_m1_plate2" origin_xyz="0 -0.024 0" origin_rpy="0 0 ${PI}" />
+    <xacro:robotis_mini_link name="${name}_upper" origin_xyz="0 0 0" origin_rpy="0 0 0" mesh_file="DMF-B04(W).stl"/>
+    <xacro:robotis_mini_revolute_joint name="${name}_m1_to_${name}_upper" parent_link="${name}_m1" child_link="${name}_upper" axis_xyz="1 0 0" origin_xyz="0 0 0" origin_rpy="${PI} ${-PI/2.0} 0" />
+    <xacro:robotis_mini_motor name="${name}_m2" origin_xyz="0 0 0" origin_rpy="0 0 0"/>
+    <xacro:robotis_mini_fixed_joint name="${name}_upper_to_${name}_m2" parent_link="${name}_upper" child_link="${name}_m2" origin_xyz="0.0 -0.045 0" origin_rpy="${PI} ${-PI/2.0} 0" />
+    <xacro:robotis_mini_link name="${name}_lower" origin_xyz="0 0 0" origin_rpy="0 0 0" mesh_file="DMF-B05(W).stl"/>
+    <xacro:robotis_mini_revolute_joint name="${name}_m2_to_${name}_lower" parent_link="${name}_m2" child_link="${name}_lower" axis_xyz="1 0 0" origin_xyz="0 0 0" origin_rpy="${-PI/2.0} ${-PI/2.0} 0" />
+    <xacro:robotis_mini_motor name="${name}_m3" origin_xyz="0 0 0" origin_rpy="0 0 0"/>
+    <xacro:robotis_mini_fixed_joint name="${name}_lower_to_${name}_m3" parent_link="${name}_lower" child_link="${name}_m3" origin_xyz="0.0 0 0" origin_rpy="0 0 0" />
   </xacro:macro>
 </robot>

File: robotis_mini_model/urdf/robotis_mini.urdf.xacro (robot description, xacro)
@@ -10,5 +10,6 @@
     <!-- <xacro:right_hand name="right_hand" parent_link="${base_link}"/> -->
     <!-- <xacro:left_hand name="left_hand" parent_link="${base_link}"/> -->
-    <!-- <xacro:leg name="right_leg" parent_link="${base_link}" xyz="0 0 0" rpy="-${0.5 * PI} ${0 * PI} ${0 * PI}" /> -->
+    <xacro:leg name="right_leg" parent_link="hip_m2_plate2" origin_xyz="0 0 0" origin_rpy="0 0 0" mirror="1.0"/>
+    <xacro:leg name="left_leg" parent_link="hip_m1_plate2" origin_xyz="0 0 0" origin_rpy="0 0 0" mirror="-1.0"/>
     <!-- <xacro:leg name="left_leg" parent_link="${base_link}" xyz="0 0 0" rpy="-${0.5 * PI} ${0 * PI} ${0 * PI}" /> -->
     <!-- <xacro:arm name="right_arm" parent_link="${base_link}" xyz="0 0 0" rpy="-${0.5 * PI} ${0 * PI} ${0 * PI}" /> -->

File: robotis_mini_model/urdf/torso.urdf.xacro (robot description, xacro)
@@ -3,10 +3,27 @@
   <xacro:include filename="$(find robotis_mini_model)/urdf/components.urdf.xacro"/>
   <xacro:macro name="torso" params="base_link">
-    <xacro:robotis_mini_link name="${base_link}" origin_xyz="0 0 0" origin_rpy="0 0 0" mesh_file="DMF-B01(W).stl"/>
-    <!--
-    <xacro:robotis_mini_link name="lower_torso_link" origin_xyz="0 0 0" origin_rpy="0 0 0" mesh_file="DMB-B02(W).stl"/>
-    <xacro:robotis_mini_fixed_joint name="${base_link}_to_lower_torso" parent_link="${base_link}" child_link="lower_torso_link" origin_xyz="0 0 0" origin_rpy="0 0 0" /> -->
+    <xacro:robotis_mini_link name="${base_link}" origin_xyz="0 0 0" origin_rpy="0 0 0" mesh_file="DMB-B02(W).stl"/>
+    <xacro:robotis_mini_link name="torso_cover" origin_xyz="0.3 0 0" origin_rpy="0 0 0" mesh_file="DMF-B01(W).stl"/>
+    <xacro:robotis_mini_fixed_joint name="${base_link}_to_torso_cover" parent_link="${base_link}" child_link="torso_cover" origin_xyz="0 0 0" origin_rpy="0 0 0" />
     <xacro:robotis_mini_motor name="shoulder_m1" origin_xyz="0 0 0" origin_rpy="0 0 0"/>
-    <xacro:robotis_mini_fixed_joint name="${base_link}_to_shoulder_m1" parent_link="${base_link}" child_link="shoulder_m1" origin_xyz="0 0 0" origin_rpy="0 0 0" /> -->
+    <xacro:robotis_mini_fixed_joint name="${base_link}_to_shoulder_m1" parent_link="${base_link}" child_link="shoulder_m1" origin_xyz="0.024 0.0415 -0.0145" origin_rpy="${-PI/2.0} 0 ${-PI/2.0}" />
+    <xacro:robotis_mini_link name="shoulder_m1_plate" origin_xyz="0 0 0" origin_rpy="0 0 0" mesh_file="SPU-5(W).stl"/>
+    <xacro:robotis_mini_fixed_joint name="shoulder_m1_to_shoulder_m1_plate" parent_link="shoulder_m1" child_link="shoulder_m1_plate" origin_xyz="0 -0.024 0" origin_rpy="0 0 ${PI}" />
+    <xacro:robotis_mini_motor name="shoulder_m2" origin_xyz="0 0 0" origin_rpy="0 0 0"/>
+    <xacro:robotis_mini_fixed_joint name="${base_link}_to_shoulder_m2" parent_link="${base_link}" child_link="shoulder_m2" origin_xyz="-0.024 0.0415 -0.0145" origin_rpy="${-PI/2.0} 0 ${PI/2.0}" />
+    <xacro:robotis_mini_link name="shoulder_m2_plate" origin_xyz="0 0 0" origin_rpy="0 0 0" mesh_file="SPU-5(W).stl"/>
+    <xacro:robotis_mini_fixed_joint name="shoulder_m2_to_shoulder_m1_plate" parent_link="shoulder_m2" child_link="shoulder_m2_plate" origin_xyz="0 -0.024 0" origin_rpy="0 0 ${PI}" />
+    <xacro:robotis_mini_motor name="hip_m1" origin_xyz="0 0 0" origin_rpy="0 0 0"/>
+    <xacro:robotis_mini_fixed_joint name="${base_link}_to_hip_m1" parent_link="${base_link}" child_link="hip_m1" origin_xyz="0.024 -0.03 -0.033" origin_rpy="0 0 ${PI}" />
+    <xacro:robotis_mini_link name="hip_m1_plate" origin_xyz="0 0 0" origin_rpy="0 0 0" mesh_file="SPU-5(W).stl"/>
+    <xacro:robotis_mini_fixed_joint name="hip_m1_to_hip_m1_plate" parent_link="hip_m1" child_link="hip_m1_plate" origin_xyz="0 -0.024 0" origin_rpy="0 0 ${PI}" />
+    <xacro:robotis_mini_link name="hip_m1_plate2" origin_xyz="0 0 0" origin_rpy="0 0 0" mesh_file="SPD-7V4(W).stl"/>
+    <xacro:robotis_mini_revolute_joint name="hip_m1_to_hip_m1_plate2" parent_link="hip_m1" child_link="hip_m1_plate2" axis_xyz="0 1 0" origin_xyz="0.0 0 0.017" origin_rpy="${PI/2.0} 0 ${PI/2.0}" />
+    <xacro:robotis_mini_motor name="hip_m2" origin_xyz="0 0 0" origin_rpy="0 0 0"/>
+    <xacro:robotis_mini_fixed_joint name="${base_link}_to_hip_m2" parent_link="${base_link}" child_link="hip_m2" origin_xyz="-0.024 -0.03 -0.033" origin_rpy="0 0 ${PI}" />
+    <xacro:robotis_mini_link name="hip_m2_plate" origin_xyz="0 0 0" origin_rpy="0 0 0" mesh_file="SPU-5(W).stl"/>
+    <xacro:robotis_mini_fixed_joint name="hip_m2_to_hip_m2_plate" parent_link="hip_m2" child_link="hip_m2_plate" origin_xyz="0 -0.024 0" origin_rpy="0 0 ${PI}" />
+    <xacro:robotis_mini_link name="hip_m2_plate2" origin_xyz="0 0 0" origin_rpy="0 0 0" mesh_file="SPD-7V4(W).stl"/>
+    <xacro:robotis_mini_revolute_joint name="hip_m2_to_hip_m2_plate2" parent_link="hip_m2" child_link="hip_m2_plate2" axis_xyz="0 1 0" origin_xyz="0.0 0 0.017" origin_rpy="${PI/2.0} 0 ${PI/2.0}" />
   </xacro:macro>
 </robot>
