Commit message: Full model

File: robotis_mini_model/urdf/arm.urdf.xacro (robot description, xacro)
@@ -2,8 +2,17 @@
 <robot xmlns:xacro="http://www.ros.org/wiki/xacro" name="robotis_mini">
   <xacro:include filename="$(find robotis_mini_model)/urdf/components.urdf.xacro"/>
-  <xacro:macro name="arm" params="name parent_link origin_xyz origin_rpy">
-    <xacro:robotis_mini_link name="${name}_upper_link" xyz="${origin_xyz}" rpy="${origin_rpy}" mesh_file="DMF-B01(W).stl"/>
-    <xacro:robotis_mini_link name="${name}_lower_link" xyz="0 0 0" rpy="0 0 0" mesh_file="DMF-B01(W).stl"/>
-    <xacro:robotis_mini_hand name="${name}_hand_link" xyz="0 0 0" rpy="0 0 0"/>
+  <xacro:macro name="arm" params="name parent_link origin_xyz origin_rpy mirror">
+    <xacro:robotis_mini_link name="${name}_shoulder" origin_xyz="${-0.012*mirror} 0 0.033" origin_rpy="${PI/2.0} 0 ${mirror*PI/2.0}" mesh_file="DMF-B03(W).stl"/>
+    <xacro:robotis_mini_revolute_joint name="${parent_link}_to_shoulder" parent_link="${parent_link}" child_link="${name}_shoulder" axis_xyz="0 0 ${mirror}" origin_xyz="0 0 0" origin_rpy="0 0 0" />
+    <xacro:robotis_mini_motor name="${name}_m1" origin_xyz="0 0 0" origin_rpy="0 0 0"/>
+    <xacro:robotis_mini_revolute_joint name="${name}_shoulder_to_${name}_m1" parent_link="${name}_shoulder" child_link="${name}_m1" axis_xyz="0 0 ${mirror}" origin_xyz="${-0.012*mirror} 0 0.033" origin_rpy="${PI/2.0} ${3*mirror*PI/4.0} 0" />
+    <xacro:robotis_mini_link name="${name}_upper" origin_xyz="0 0 0" origin_rpy="0 0 0" mesh_file="DMF-B04(W).stl"/>
+    <xacro:robotis_mini_fixed_joint name="${name}_m1_to_${name}_upper" parent_link="${name}_m1" child_link="${name}_upper" origin_xyz="0 -0.045 0" origin_rpy="${PI} ${(1.0*mirror)*PI/2.0} 0" />
+    <xacro:robotis_mini_motor name="${name}_m2" origin_xyz="0 0 0" origin_rpy="0 0 0"/>
+    <xacro:robotis_mini_revolute_joint name="${name}_upper_to_${name}_m2" parent_link="${name}_upper" child_link="${name}_m2" axis_xyz="0 0 ${mirror}" origin_xyz="0 0 0.0" origin_rpy="0 ${mirror*PI/2.0} ${PI}" />
+    <xacro:robotis_mini_link name="${name}_m2_plate" origin_xyz="0 0 0" origin_rpy="0 0 0" mesh_file="SPU-5(W).stl"/>
+    <xacro:robotis_mini_fixed_joint name="${name}_m2_to_${name}_m2_plate" parent_link="${name}_m2" child_link="${name}_m2_plate" origin_xyz="0 -0.024 0" origin_rpy="0 0 ${PI}" />
+    <xacro:robotis_mini_link name="${name}_m2_plate2" origin_xyz="0 0 0" origin_rpy="0 0 0" mesh_file="SPD-3B3(W).stl"/>
+    <xacro:robotis_mini_fixed_joint name="${name}_m2_to_${name}_m2_plate2" parent_link="${name}_m2" child_link="${name}_m2_plate2" origin_xyz="0 -0.028 0" origin_rpy="0 0 ${PI}" />
   </xacro:macro>
 </robot>

File: robotis_mini_model/urdf/left_hand.urdf.xacro (robot description, xacro)
@@ -4,5 +4,5 @@
   <xacro:macro name="left_hand" params="name parent_link">
     <xacro:robotis_mini_link name="${name}_l1" origin_xyz="0 0 0" origin_rpy="0 0 0" mesh_file="SPO-5(GR).stl"/>
-    <xacro:robotis_mini_fixed_joint name="${parent_link}_to_{name}_l1" parent_link="${parent_link}" child_link="${name}_l1" origin_xyz="0.1 0 0" origin_rpy="0 0 0" />
+    <xacro:robotis_mini_fixed_joint name="${parent_link}_to_{name}_l1" parent_link="${parent_link}" child_link="${name}_l1" origin_xyz="0 0.002 0" origin_rpy="0 ${PI/2.0} 0" />
     <xacro:robotis_mini_link name="${name}_l2" origin_xyz="0 0 0" origin_rpy="0 0 0" mesh_file="SPO-5(GR).stl"/>
     <xacro:robotis_mini_fixed_joint name="${name}_l1_to_{name}_l2" parent_link="${name}_l1" child_link="${name}_l2" origin_xyz="0 0.003 0" origin_rpy="0 0 0" />

File: robotis_mini_model/urdf/leg.urdf.xacro (robot description, xacro)
@@ -4,11 +4,11 @@
   <xacro:macro name="leg" params="name parent_link origin_xyz origin_rpy mirror">
     <xacro:robotis_mini_link name="${name}_m1_plate" origin_xyz="${origin_xyz}" origin_rpy="${origin_rpy}" mesh_file="SPD-3B5(W).stl"/>
-    <xacro:robotis_mini_revolute_joint name="${parent_link}_to_${name}_m1_plate" parent_link="${parent_link}" child_link="${name}_m1_plate" axis_xyz="0 1 0" origin_xyz="0 0.1 0" origin_rpy="0 0 0" />
+    <xacro:robotis_mini_fixed_joint name="${parent_link}_to_${name}_m1_plate" parent_link="${parent_link}" child_link="${name}_m1_plate" origin_xyz="0 0.003 0" origin_rpy="0 ${PI} 0" />
     <xacro:robotis_mini_motor name="${name}_m1" origin_xyz="0 0 0" origin_rpy="0 0 0"/>
-    <xacro:robotis_mini_fixed_joint name="${name}_m1_plate_to_${name}_m1" parent_link="${name}_m1_plate" child_link="${name}_m1" origin_xyz="0.012 0.013 0" origin_rpy="${PI} ${PI} ${-PI/2.0}" />
+    <xacro:robotis_mini_fixed_joint name="${name}_m1_plate_to_${name}_m1" parent_link="${name}_m1_plate" child_link="${name}_m1" origin_xyz="-0.006 0.013 0" origin_rpy="${(mirror/2.0 + 0.5)*PI} ${PI} ${(-1.0*mirror)*PI/2.0}" />
     <xacro:robotis_mini_link name="${name}_m1_plate2" origin_xyz="0 0 0" origin_rpy="0 0 0" mesh_file="SPU-5(W).stl"/>
     <xacro:robotis_mini_fixed_joint name="${name}_m1_to_${name}_m1_plate2" parent_link="${name}_m1" child_link="${name}_m1_plate2" origin_xyz="0 -0.024 0" origin_rpy="0 0 ${PI}" />
     <xacro:robotis_mini_link name="${name}_upper" origin_xyz="0 0 0" origin_rpy="0 0 0" mesh_file="DMF-B04(W).stl"/>
-    <xacro:robotis_mini_revolute_joint name="${name}_m1_to_${name}_upper" parent_link="${name}_m1" child_link="${name}_upper" axis_xyz="1 0 0" origin_xyz="0 0 0" origin_rpy="${PI} ${-PI/2.0} 0" />
+    <xacro:robotis_mini_revolute_joint name="${name}_m1_to_${name}_upper" parent_link="${name}_m1" child_link="${name}_upper" axis_xyz="1 0 0" origin_xyz="0 0 0" origin_rpy="${PI} ${(-1.0*mirror)*PI/2.0} 0" />
     <xacro:robotis_mini_motor name="${name}_m2" origin_xyz="0 0 0" origin_rpy="0 0 0"/>
     <xacro:robotis_mini_fixed_joint name="${name}_upper_to_${name}_m2" parent_link="${name}_upper" child_link="${name}_m2" origin_xyz="0.0 -0.045 0" origin_rpy="${PI} ${-PI/2.0} 0" />
@@ -16,5 +16,15 @@
     <xacro:robotis_mini_revolute_joint name="${name}_m2_to_${name}_lower" parent_link="${name}_m2" child_link="${name}_lower" axis_xyz="1 0 0" origin_xyz="0 0 0" origin_rpy="${-PI/2.0} ${-PI/2.0} 0" />
     <xacro:robotis_mini_motor name="${name}_m3" origin_xyz="0 0 0" origin_rpy="0 0 0"/>
-    <xacro:robotis_mini_fixed_joint name="${name}_lower_to_${name}_m3" parent_link="${name}_lower" child_link="${name}_m3" origin_xyz="0.0 0 0" origin_rpy="0 0 0" />
+    <xacro:robotis_mini_revolute_joint name="${name}_lower_to_${name}_m3" parent_link="${name}_lower" child_link="${name}_m3" axis_xyz="0 0 ${mirror}" origin_xyz="0.0 0 0.042" origin_rpy="${PI/2.0} 0 ${mirror*PI/2.0}" />
+    <xacro:robotis_mini_link name="${name}_m3_plate1" origin_xyz="0 0 0" origin_rpy="0 0 0"  mesh_file="SPD-3B7(W).stl"/>
+    <xacro:robotis_mini_fixed_joint name="${name}_m3_to_${name}_m3_plate1" parent_link="${name}_m3" child_link="${name}_m3_plate1" origin_xyz="${-mirror*0.012} -0.006 0" origin_rpy="0 0 ${PI/2.0}" />
+    <xacro:robotis_mini_link name="${name}_m3_plate2" origin_xyz="0 0 0" origin_rpy="0 0 0"  mesh_file="SPD-3B5(W).stl"/>
+    <xacro:robotis_mini_fixed_joint name="${name}_m3_to_${name}_m3_plate2" parent_link="${name}_m3" child_link="${name}_m3_plate2" origin_xyz="${-mirror*0.015} 0 0" origin_rpy="0 0 ${PI/2.0}" />
+    <xacro:robotis_mini_motor name="${name}_m4" origin_xyz="0 0 0" origin_rpy="0 0 0"/>
+    <xacro:robotis_mini_revolute_joint name="${name}_m3_to_${name}_m4" parent_link="${name}_m3" child_link="${name}_m4" axis_xyz="0 0 ${-mirror}" origin_xyz="${-mirror*0.032} 0 0" origin_rpy="${PI/2.0} 0 ${mirror*PI/2.0}" />
+    <xacro:robotis_mini_link name="${name}_foot" origin_xyz="0 0 0" origin_rpy="0 0 0"  mesh_file="DMF-B06(W).stl"/>
+    <xacro:robotis_mini_fixed_joint name="${name}_m4_to_${name}_foot" parent_link="${name}_m4" child_link="${name}_foot" origin_xyz="${mirror*0.03} -0.009 0" origin_rpy="0 0 ${mirror*PI/2.0}" />
+    <xacro:robotis_mini_link name="${name}_foot_sole" origin_xyz="0 0 0" origin_rpy="0 0 0"  mesh_file="DMF-B07(GR).stl"/>
+    <xacro:robotis_mini_fixed_joint name="${name}_foot_to_${name}_foot_sole" parent_link="${name}_foot" child_link="${name}_foot_sole" origin_xyz="0 0 0.03" origin_rpy="0 0 0" />
   </xacro:macro>
 </robot>

File: robotis_mini_model/urdf/right_hand.urdf.xacro (robot description, xacro)
@@ -4,5 +4,5 @@
   <xacro:macro name="right_hand" params="name parent_link">
     <xacro:robotis_mini_link name="${name}_l1" origin_xyz="0 0 0" origin_rpy="0 0 0" mesh_file="SPO-5(GR).stl"/>
-    <xacro:robotis_mini_fixed_joint name="${parent_link}_to_{name}_l2" parent_link="${parent_link}" child_link="${name}_l1" origin_xyz="0.1 0 0" origin_rpy="0 0 0" />
+    <xacro:robotis_mini_fixed_joint name="${parent_link}_to_{name}_l2" parent_link="${parent_link}" child_link="${name}_l1" origin_xyz="0 0 0" origin_rpy="0 ${-PI/2.0} 0" />
     <xacro:robotis_mini_link name="${name}_l2" origin_xyz="0 0 0" origin_rpy="0 0 0" mesh_file="SPO-5(GR).stl"/>
     <xacro:robotis_mini_fixed_joint name="${name}_l1_to_{name}_l2" parent_link="${name}_l1" child_link="${name}_l2" origin_xyz="0 0.003 0" origin_rpy="0 0 0" />

File: robotis_mini_model/urdf/robotis_mini.urdf.xacro (robot description, xacro)
@@ -8,10 +8,9 @@
     <xacro:property name="base_link" value="torso_link" />
     <xacro:torso base_link="${base_link}"/>
-    <!-- <xacro:right_hand name="right_hand" parent_link="${base_link}"/> -->
-    <!-- <xacro:left_hand name="left_hand" parent_link="${base_link}"/> -->
     <xacro:leg name="right_leg" parent_link="hip_m2_plate2" origin_xyz="0 0 0" origin_rpy="0 0 0" mirror="1.0"/>
     <xacro:leg name="left_leg" parent_link="hip_m1_plate2" origin_xyz="0 0 0" origin_rpy="0 0 0" mirror="-1.0"/>
-    <!-- <xacro:leg name="left_leg" parent_link="${base_link}" xyz="0 0 0" rpy="-${0.5 * PI} ${0 * PI} ${0 * PI}" /> -->
-    <!-- <xacro:arm name="right_arm" parent_link="${base_link}" xyz="0 0 0" rpy="-${0.5 * PI} ${0 * PI} ${0 * PI}" /> -->
-    <!-- <xacro:arm name="right_arm" parent_link="${base_link}" xyz="0 0 0" rpy="-${0.5 * PI} ${0 * PI} ${0 * PI}" /> -->
+    <xacro:arm name="right_arm" parent_link="shoulder_m2" origin_xyz="0 0 0" origin_rpy="-${0.5 * PI} ${0 * PI} ${0 * PI}" mirror="1" />
+    <xacro:arm name="left_arm" parent_link="shoulder_m1" origin_xyz="0 0 0" origin_rpy="-${0.5 * PI} ${0 * PI} ${0 * PI}" mirror="-1" />
+    <xacro:right_hand name="right_hand" parent_link="right_arm_m2_plate2"/>
+    <xacro:left_hand name="left_hand" parent_link="left_arm_m2_plate2"/>
 </robot>

File: robotis_mini_model/urdf/torso.urdf.xacro (robot description, xacro)
@@ -4,6 +4,10 @@
   <xacro:macro name="torso" params="base_link">
     <xacro:robotis_mini_link name="${base_link}" origin_xyz="0 0 0" origin_rpy="0 0 0" mesh_file="DMB-B02(W).stl"/>
-    <xacro:robotis_mini_link name="torso_cover" origin_xyz="0.3 0 0" origin_rpy="0 0 0" mesh_file="DMF-B01(W).stl"/>
-    <xacro:robotis_mini_fixed_joint name="${base_link}_to_torso_cover" parent_link="${base_link}" child_link="torso_cover" origin_xyz="0 0 0" origin_rpy="0 0 0" />
+    <xacro:robotis_mini_link name="torso_cover" origin_xyz="0 0 0" origin_rpy="0 0 0" mesh_file="DMF-B01(W).stl"/>
+    <xacro:robotis_mini_fixed_joint name="${base_link}_to_torso_cover" parent_link="${base_link}" child_link="torso_cover" origin_xyz="0 0.04 -0.01" origin_rpy="0 0 0" />
+    <xacro:robotis_mini_motor name="head_m" origin_xyz="0 0 0" origin_rpy="0 0 0"/>
+    <xacro:robotis_mini_fixed_joint name="$torso_cover_to_head_m" parent_link="torso_cover" child_link="head_m" origin_xyz="0 0.036 0.005" origin_rpy="${PI/2.0} ${PI} 0" />
+    <xacro:robotis_mini_link name="head" origin_xyz="0 0 0" origin_rpy="0 0 0" mesh_file="DMF-F01(W).stl"/>
+    <xacro:robotis_mini_fixed_joint name="$head_m_to_head" parent_link="head_m" child_link="head" origin_xyz="0.0 -0.021 0.002" origin_rpy="${-PI/2.0} 0 ${PI}" />
     <xacro:robotis_mini_motor name="shoulder_m1" origin_xyz="0 0 0" origin_rpy="0 0 0"/>
     <xacro:robotis_mini_fixed_joint name="${base_link}_to_shoulder_m1" parent_link="${base_link}" child_link="shoulder_m1" origin_xyz="0.024 0.0415 -0.0145" origin_rpy="${-PI/2.0} 0 ${-PI/2.0}" />
@@ -25,5 +29,5 @@
     <xacro:robotis_mini_fixed_joint name="hip_m2_to_hip_m2_plate" parent_link="hip_m2" child_link="hip_m2_plate" origin_xyz="0 -0.024 0" origin_rpy="0 0 ${PI}" />
     <xacro:robotis_mini_link name="hip_m2_plate2" origin_xyz="0 0 0" origin_rpy="0 0 0" mesh_file="SPD-7V4(W).stl"/>
-    <xacro:robotis_mini_revolute_joint name="hip_m2_to_hip_m2_plate2" parent_link="hip_m2" child_link="hip_m2_plate2" axis_xyz="0 1 0" origin_xyz="0.0 0 0.017" origin_rpy="${PI/2.0} 0 ${PI/2.0}" />
+    <xacro:robotis_mini_revolute_joint name="hip_m2_to_hip_m2_plate2" parent_link="hip_m2" child_link="hip_m2_plate2" axis_xyz="0 -1 0" origin_xyz="0.0 0 0.017" origin_rpy="${PI/2.0} 0 ${PI/2.0}" />
   </xacro:macro>
 </robot>

Commit message: urdf

File: robotis_mini_model/urdf/arm.urdf.xacro (robot description, xacro)
@@ -2,5 +2,5 @@
 <robot xmlns:xacro="http://www.ros.org/wiki/xacro" name="robotis_mini">
   <xacro:include filename="$(find robotis_mini_model)/urdf/components.urdf.xacro"/>
-  <xacro:macro name="arm" params="name parent_link origin_xyz origin_rpy mirror">
+  <xacro:macro name="arm" params="name parent_link mirror">
     <xacro:robotis_mini_link name="${name}_shoulder" origin_xyz="${-0.012*mirror} 0 0.033" origin_rpy="${PI/2.0} 0 ${mirror*PI/2.0}" mesh_file="DMF-B03(W).stl"/>
     <xacro:robotis_mini_revolute_joint name="${parent_link}_to_shoulder" parent_link="${parent_link}" child_link="${name}_shoulder" axis_xyz="0 0 ${mirror}" origin_xyz="0 0 0" origin_rpy="0 0 0" />

File: robotis_mini_model/urdf/leg.urdf.xacro (robot description, xacro)
@@ -2,6 +2,6 @@
 <robot xmlns:xacro="http://www.ros.org/wiki/xacro" name="robotis_mini">
   <xacro:include filename="$(find robotis_mini_model)/urdf/components.urdf.xacro"/>
-  <xacro:macro name="leg" params="name parent_link origin_xyz origin_rpy mirror">
-    <xacro:robotis_mini_link name="${name}_m1_plate" origin_xyz="${origin_xyz}" origin_rpy="${origin_rpy}" mesh_file="SPD-3B5(W).stl"/>
+  <xacro:macro name="leg" params="name parent_link mirror">
+    <xacro:robotis_mini_link name="${name}_m1_plate" origin_xyz="0 0 0" origin_rpy="0 0 0" mesh_file="SPD-3B5(W).stl"/>
     <xacro:robotis_mini_fixed_joint name="${parent_link}_to_${name}_m1_plate" parent_link="${parent_link}" child_link="${name}_m1_plate" origin_xyz="0 0.003 0" origin_rpy="0 ${PI} 0" />
     <xacro:robotis_mini_motor name="${name}_m1" origin_xyz="0 0 0" origin_rpy="0 0 0"/>

File: robotis_mini_model/urdf/robotis_mini.urdf.xacro (robot description, xacro)
@@ -8,8 +8,8 @@
     <xacro:property name="base_link" value="torso_link" />
     <xacro:torso base_link="${base_link}"/>
-    <xacro:leg name="right_leg" parent_link="hip_m2_plate2" origin_xyz="0 0 0" origin_rpy="0 0 0" mirror="1.0"/>
-    <xacro:leg name="left_leg" parent_link="hip_m1_plate2" origin_xyz="0 0 0" origin_rpy="0 0 0" mirror="-1.0"/>
-    <xacro:arm name="right_arm" parent_link="shoulder_m2" origin_xyz="0 0 0" origin_rpy="-${0.5 * PI} ${0 * PI} ${0 * PI}" mirror="1" />
-    <xacro:arm name="left_arm" parent_link="shoulder_m1" origin_xyz="0 0 0" origin_rpy="-${0.5 * PI} ${0 * PI} ${0 * PI}" mirror="-1" />
+    <xacro:leg name="right_leg" parent_link="hip_m2_plate2" mirror="1.0"/>
+    <xacro:leg name="left_leg" parent_link="hip_m1_plate2" mirror="-1.0"/>
+    <xacro:arm name="right_arm" parent_link="shoulder_m2" mirror="1.0" />
+    <xacro:arm name="left_arm" parent_link="shoulder_m1" mirror="-1.0" />
     <xacro:right_hand name="right_hand" parent_link="right_arm_m2_plate2"/>
     <xacro:left_hand name="left_hand" parent_link="left_arm_m2_plate2"/>
