Commit message: Working version of a node that uses pypot to read the motors and publish them to ros and the ros side moves the urdf model accordingly

File: robotis_mini_ros/urdf/arm.urdf.xacro (robot description, xacro)
@@ -1,18 +1,18 @@
 <?xml version="1.0"?>
 <robot xmlns:xacro="http://www.ros.org/wiki/xacro" name="robotis_mini">
-  <xacro:include filename="$(find robotis_mini_model)/urdf/components.urdf.xacro"/>
+  <xacro:include filename="$(find robotis_mini_ros)/urdf/components.urdf.xacro"/>
   <xacro:macro name="arm" params="name parent_link mirror">
     <xacro:robotis_mini_link name="${name}_shoulder" origin_xyz="${-0.012*mirror} 0 0.033" origin_rpy="${PI/2.0} 0 ${mirror*PI/2.0}" mesh_file="DMF-B03(W).stl"/>
-    <xacro:robotis_mini_revolute_joint name="${parent_link}_to_shoulder" parent_link="${parent_link}" child_link="${name}_shoulder" axis_xyz="0 0 ${mirror}" origin_xyz="0 0 0" origin_rpy="0 0 0" />
-    <xacro:robotis_mini_motor name="${name}_m1" origin_xyz="0 0 0" origin_rpy="0 0 0"/>
-    <xacro:robotis_mini_revolute_joint name="${name}_shoulder_to_${name}_m1" parent_link="${name}_shoulder" child_link="${name}_m1" axis_xyz="0 0 ${mirror}" origin_xyz="${-0.012*mirror} 0 0.033" origin_rpy="${PI/2.0} ${3*mirror*PI/4.0} 0" />
-    <xacro:robotis_mini_link name="${name}_upper" origin_xyz="0 0 0" origin_rpy="0 0 0" mesh_file="DMF-B04(W).stl"/>
-    <xacro:robotis_mini_fixed_joint name="${name}_m1_to_${name}_upper" parent_link="${name}_m1" child_link="${name}_upper" origin_xyz="0 -0.045 0" origin_rpy="${PI} ${(1.0*mirror)*PI/2.0} 0" />
-    <xacro:robotis_mini_motor name="${name}_m2" origin_xyz="0 0 0" origin_rpy="0 0 0"/>
-    <xacro:robotis_mini_revolute_joint name="${name}_upper_to_${name}_m2" parent_link="${name}_upper" child_link="${name}_m2" axis_xyz="0 0 ${mirror}" origin_xyz="0 0 0.0" origin_rpy="0 ${mirror*PI/2.0} ${PI}" />
-    <xacro:robotis_mini_link name="${name}_m2_plate" origin_xyz="0 0 0" origin_rpy="0 0 0" mesh_file="SPU-5(W).stl"/>
-    <xacro:robotis_mini_fixed_joint name="${name}_m2_to_${name}_m2_plate" parent_link="${name}_m2" child_link="${name}_m2_plate" origin_xyz="0 -0.024 0" origin_rpy="0 0 ${PI}" />
-    <xacro:robotis_mini_link name="${name}_m2_plate2" origin_xyz="0 0 0" origin_rpy="0 0 0" mesh_file="SPD-3B3(W).stl"/>
-    <xacro:robotis_mini_fixed_joint name="${name}_m2_to_${name}_m2_plate2" parent_link="${name}_m2" child_link="${name}_m2_plate2" origin_xyz="0 -0.028 0" origin_rpy="0 0 ${PI}" />
+    <xacro:robotis_mini_revolute_joint name="${name}_shoulder1" parent_link="${parent_link}" child_link="${name}_shoulder" axis_xyz="0 0 ${mirror}" origin_xyz="0 0 0" origin_rpy="0 0 0" />
+    <xacro:robotis_mini_motor name="${name}_arm_m1" origin_xyz="0 0 0" origin_rpy="0 0 0"/>
+    <xacro:robotis_mini_revolute_joint name="${name}_shoulder2" parent_link="${name}_shoulder" child_link="${name}_arm_m1" axis_xyz="0 0 ${mirror}" origin_xyz="${-0.012*mirror} 0 0.033" origin_rpy="${PI/2.0} ${PI} 0" />
+    <xacro:robotis_mini_link name="${name}_arm_upper" origin_xyz="0 0 0" origin_rpy="0 0 0" mesh_file="DMF-B04(W).stl"/>
+    <xacro:robotis_mini_fixed_joint name="${name}_arm_m1_to_${name}_arm_upper" parent_link="${name}_arm_m1" child_link="${name}_arm_upper" origin_xyz="0 -0.045 0" origin_rpy="${PI} ${(1.0*mirror)*PI/2.0} 0" />
+    <xacro:robotis_mini_motor name="${name}_arm_m2" origin_xyz="0 0 0" origin_rpy="0 0 0"/>
+    <xacro:robotis_mini_revolute_joint name="${name}_elbow" parent_link="${name}_arm_upper" child_link="${name}_arm_m2" axis_xyz="0 0 ${mirror}" origin_xyz="0 0 0.0" origin_rpy="0 ${mirror*PI/2.0} ${PI}" />
+    <xacro:robotis_mini_link name="${name}_arm_m2_plate" origin_xyz="0 0 0" origin_rpy="0 0 0" mesh_file="SPU-5(W).stl"/>
+    <xacro:robotis_mini_fixed_joint name="${name}_arm_m2_to_${name}_arm_m2_plate" parent_link="${name}_arm_m2" child_link="${name}_arm_m2_plate" origin_xyz="0 -0.024 0" origin_rpy="0 0 ${PI}" />
+    <xacro:robotis_mini_link name="${name}_arm_m2_plate2" origin_xyz="0 0 0" origin_rpy="0 0 0" mesh_file="SPD-3B3(W).stl"/>
+    <xacro:robotis_mini_fixed_joint name="${name}_arm_m2_to_${name}_arm_m2_plate2" parent_link="${name}_arm_m2" child_link="${name}_arm_m2_plate2" origin_xyz="0 -0.028 0" origin_rpy="0 0 ${PI}" />
   </xacro:macro>
 </robot>

File: robotis_mini_ros/urdf/components.urdf.xacro (robot description, xacro)
@@ -17,5 +17,5 @@
         <origin xyz="${origin_xyz}" rpy="${origin_rpy}" />
         <geometry>
-          <mesh filename="package://robotis_mini_model/meshes/${mesh_file}" scale="0.001 0.001 0.001" />
+          <mesh filename="package://robotis_mini_ros/meshes/${mesh_file}" scale="0.001 0.001 0.001" />
         </geometry>
         <xacro:robotis_mini_material/>
@@ -28,5 +28,5 @@
         <origin xyz="${origin_xyz}" rpy="${origin_rpy}" />
         <geometry>
-          <mesh filename="package://robotis_mini_model/meshes/XL-320D.stl" scale="0.001 0.001 0.001" />
+          <mesh filename="package://robotis_mini_ros/meshes/XL-320D.stl" scale="0.001 0.001 0.001" />
         </geometry>
         <xacro:robotis_mini_motor_material/>

File: robotis_mini_ros/urdf/left_hand.urdf.xacro (robot description, xacro)
@@ -1,5 +1,5 @@
 <?xml version="1.0"?>
 <robot xmlns:xacro="http://www.ros.org/wiki/xacro" name="robotis_mini">
-  <xacro:include filename="$(find robotis_mini_model)/urdf/components.urdf.xacro"/>
+  <xacro:include filename="$(find robotis_mini_ros)/urdf/components.urdf.xacro"/>
   <xacro:macro name="left_hand" params="name parent_link">
     <xacro:robotis_mini_link name="${name}_l1" origin_xyz="0 0 0" origin_rpy="0 0 0" mesh_file="SPO-5(GR).stl"/>

File: robotis_mini_ros/urdf/leg.urdf.xacro (robot description, xacro)
@@ -1,5 +1,5 @@
 <?xml version="1.0"?>
 <robot xmlns:xacro="http://www.ros.org/wiki/xacro" name="robotis_mini">
-  <xacro:include filename="$(find robotis_mini_model)/urdf/components.urdf.xacro"/>
+  <xacro:include filename="$(find robotis_mini_ros)/urdf/components.urdf.xacro"/>
   <xacro:macro name="leg" params="name parent_link mirror">
     <xacro:robotis_mini_link name="${name}_m1_plate" origin_xyz="0 0 0" origin_rpy="0 0 0" mesh_file="SPD-3B5(W).stl"/>
@@ -10,11 +10,11 @@
     <xacro:robotis_mini_fixed_joint name="${name}_m1_to_${name}_m1_plate2" parent_link="${name}_m1" child_link="${name}_m1_plate2" origin_xyz="0 -0.024 0" origin_rpy="0 0 ${PI}" />
     <xacro:robotis_mini_link name="${name}_upper" origin_xyz="0 0 0" origin_rpy="0 0 0" mesh_file="DMF-B04(W).stl"/>
-    <xacro:robotis_mini_revolute_joint name="${name}_m1_to_${name}_upper" parent_link="${name}_m1" child_link="${name}_upper" axis_xyz="1 0 0" origin_xyz="0 0 0" origin_rpy="${PI} ${(-1.0*mirror)*PI/2.0} 0" />
+    <xacro:robotis_mini_revolute_joint name="${name}_hip2" parent_link="${name}_m1" child_link="${name}_upper" axis_xyz="1 0 0" origin_xyz="0 0 0" origin_rpy="${PI} ${(-1.0*mirror)*PI/2.0} 0" />
     <xacro:robotis_mini_motor name="${name}_m2" origin_xyz="0 0 0" origin_rpy="0 0 0"/>
     <xacro:robotis_mini_fixed_joint name="${name}_upper_to_${name}_m2" parent_link="${name}_upper" child_link="${name}_m2" origin_xyz="0.0 -0.045 0" origin_rpy="${PI} ${-PI/2.0} 0" />
     <xacro:robotis_mini_link name="${name}_lower" origin_xyz="0 0 0" origin_rpy="0 0 0" mesh_file="DMF-B05(W).stl"/>
-    <xacro:robotis_mini_revolute_joint name="${name}_m2_to_${name}_lower" parent_link="${name}_m2" child_link="${name}_lower" axis_xyz="1 0 0" origin_xyz="0 0 0" origin_rpy="${-PI/2.0} ${-PI/2.0} 0" />
+    <xacro:robotis_mini_revolute_joint name="${name}_knee" parent_link="${name}_m2" child_link="${name}_lower" axis_xyz="1 0 0" origin_xyz="0 0 0" origin_rpy="${-PI/2.0} ${-PI/2.0} 0" />
     <xacro:robotis_mini_motor name="${name}_m3" origin_xyz="0 0 0" origin_rpy="0 0 0"/>
-    <xacro:robotis_mini_revolute_joint name="${name}_lower_to_${name}_m3" parent_link="${name}_lower" child_link="${name}_m3" axis_xyz="0 0 ${mirror}" origin_xyz="0.0 0 0.042" origin_rpy="${PI/2.0} 0 ${mirror*PI/2.0}" />
+    <xacro:robotis_mini_revolute_joint name="${name}_ankle1" parent_link="${name}_lower" child_link="${name}_m3" axis_xyz="0 0 ${mirror}" origin_xyz="0.0 0 0.042" origin_rpy="${PI/2.0} 0 ${mirror*PI/2.0}" />
     <xacro:robotis_mini_link name="${name}_m3_plate1" origin_xyz="0 0 0" origin_rpy="0 0 0"  mesh_file="SPD-3B7(W).stl"/>
     <xacro:robotis_mini_fixed_joint name="${name}_m3_to_${name}_m3_plate1" parent_link="${name}_m3" child_link="${name}_m3_plate1" origin_xyz="${-mirror*0.012} -0.006 0" origin_rpy="0 0 ${PI/2.0}" />
@@ -22,5 +22,5 @@
     <xacro:robotis_mini_fixed_joint name="${name}_m3_to_${name}_m3_plate2" parent_link="${name}_m3" child_link="${name}_m3_plate2" origin_xyz="${-mirror*0.015} 0 0" origin_rpy="0 0 ${PI/2.0}" />
     <xacro:robotis_mini_motor name="${name}_m4" origin_xyz="0 0 0" origin_rpy="0 0 0"/>
-    <xacro:robotis_mini_revolute_joint name="${name}_m3_to_${name}_m4" parent_link="${name}_m3" child_link="${name}_m4" axis_xyz="0 0 ${-mirror}" origin_xyz="${-mirror*0.032} 0 0" origin_rpy="${PI/2.0} 0 ${mirror*PI/2.0}" />
+    <xacro:robotis_mini_revolute_joint name="${name}_ankle2" parent_link="${name}_m3" child_link="${name}_m4" axis_xyz="0 0 ${-mirror}" origin_xyz="${-mirror*0.032} 0 0" origin_rpy="${PI/2.0} 0 ${mirror*PI/2.0}" />
     <xacro:robotis_mini_link name="${name}_foot" origin_xyz="0 0 0" origin_rpy="0 0 0"  mesh_file="DMF-B06(W).stl"/>
     <xacro:robotis_mini_fixed_joint name="${name}_m4_to_${name}_foot" parent_link="${name}_m4" child_link="${name}_foot" origin_xyz="${mirror*0.03} -0.009 0" origin_rpy="0 0 ${mirror*PI/2.0}" />

File: robotis_mini_ros/urdf/right_hand.urdf.xacro (robot description, xacro)
@@ -1,5 +1,5 @@
 <?xml version="1.0"?>
 <robot xmlns:xacro="http://www.ros.org/wiki/xacro" name="robotis_mini">
-  <xacro:include filename="$(find robotis_mini_model)/urdf/components.urdf.xacro"/>
+  <xacro:include filename="$(find robotis_mini_ros)/urdf/components.urdf.xacro"/>
   <xacro:macro name="right_hand" params="name parent_link">
     <xacro:robotis_mini_link name="${name}_l1" origin_xyz="0 0 0" origin_rpy="0 0 0" mesh_file="SPO-5(GR).stl"/>

File: robotis_mini_ros/urdf/robotis_mini.urdf.xacro (robot description, xacro)
@@ -1,15 +1,15 @@
 <?xml version="1.0"?>
 <robot xmlns:xacro="http://www.ros.org/wiki/xacro" name="robotis_mini">
-    <xacro:include filename="$(find robotis_mini_model)/urdf/leg.urdf.xacro"/>
-    <xacro:include filename="$(find robotis_mini_model)/urdf/arm.urdf.xacro"/>
-    <xacro:include filename="$(find robotis_mini_model)/urdf/torso.urdf.xacro"/>
-    <xacro:include filename="$(find robotis_mini_model)/urdf/right_hand.urdf.xacro"/>
-    <xacro:include filename="$(find robotis_mini_model)/urdf/left_hand.urdf.xacro"/>
+    <xacro:include filename="$(find robotis_mini_ros)/urdf/leg.urdf.xacro"/>
+    <xacro:include filename="$(find robotis_mini_ros)/urdf/arm.urdf.xacro"/>
+    <xacro:include filename="$(find robotis_mini_ros)/urdf/torso.urdf.xacro"/>
+    <xacro:include filename="$(find robotis_mini_ros)/urdf/right_hand.urdf.xacro"/>
+    <xacro:include filename="$(find robotis_mini_ros)/urdf/left_hand.urdf.xacro"/>
     <xacro:property name="base_link" value="torso_link" />
     <xacro:torso base_link="${base_link}"/>
-    <xacro:leg name="right_leg" parent_link="hip_m2_plate2" mirror="1.0"/>
-    <xacro:leg name="left_leg" parent_link="hip_m1_plate2" mirror="-1.0"/>
-    <xacro:arm name="right_arm" parent_link="shoulder_m2" mirror="1.0" />
-    <xacro:arm name="left_arm" parent_link="shoulder_m1" mirror="-1.0" />
+    <xacro:leg name="right" parent_link="hip_m2_plate2" mirror="1.0"/>
+    <xacro:leg name="left" parent_link="hip_m1_plate2" mirror="-1.0"/>
+    <xacro:arm name="right" parent_link="shoulder_m2" mirror="1.0" />
+    <xacro:arm name="left" parent_link="shoulder_m1" mirror="-1.0" />
     <xacro:right_hand name="right_hand" parent_link="right_arm_m2_plate2"/>
     <xacro:left_hand name="left_hand" parent_link="left_arm_m2_plate2"/>

File: robotis_mini_ros/urdf/torso.urdf.xacro (robot description, xacro)
@@ -1,5 +1,5 @@
 <?xml version="1.0"?>
 <robot xmlns:xacro="http://www.ros.org/wiki/xacro" name="robotis_mini">
-  <xacro:include filename="$(find robotis_mini_model)/urdf/components.urdf.xacro"/>
+  <xacro:include filename="$(find robotis_mini_ros)/urdf/components.urdf.xacro"/>
   <xacro:macro name="torso" params="base_link">
     <xacro:robotis_mini_link name="${base_link}" origin_xyz="0 0 0" origin_rpy="0 0 0" mesh_file="DMB-B02(W).stl"/>
@@ -23,5 +23,5 @@
     <xacro:robotis_mini_fixed_joint name="hip_m1_to_hip_m1_plate" parent_link="hip_m1" child_link="hip_m1_plate" origin_xyz="0 -0.024 0" origin_rpy="0 0 ${PI}" />
     <xacro:robotis_mini_link name="hip_m1_plate2" origin_xyz="0 0 0" origin_rpy="0 0 0" mesh_file="SPD-7V4(W).stl"/>
-    <xacro:robotis_mini_revolute_joint name="hip_m1_to_hip_m1_plate2" parent_link="hip_m1" child_link="hip_m1_plate2" axis_xyz="0 1 0" origin_xyz="0.0 0 0.017" origin_rpy="${PI/2.0} 0 ${PI/2.0}" />
+    <xacro:robotis_mini_revolute_joint name="left_hip1" parent_link="hip_m1" child_link="hip_m1_plate2" axis_xyz="0 1 0" origin_xyz="0.0 0 0.017" origin_rpy="${PI/2.0} 0 ${PI/2.0}" />
     <xacro:robotis_mini_motor name="hip_m2" origin_xyz="0 0 0" origin_rpy="0 0 0"/>
     <xacro:robotis_mini_fixed_joint name="${base_link}_to_hip_m2" parent_link="${base_link}" child_link="hip_m2" origin_xyz="-0.024 -0.03 -0.033" origin_rpy="0 0 ${PI}" />
@@ -29,5 +29,5 @@
     <xacro:robotis_mini_fixed_joint name="hip_m2_to_hip_m2_plate" parent_link="hip_m2" child_link="hip_m2_plate" origin_xyz="0 -0.024 0" origin_rpy="0 0 ${PI}" />
     <xacro:robotis_mini_link name="hip_m2_plate2" origin_xyz="0 0 0" origin_rpy="0 0 0" mesh_file="SPD-7V4(W).stl"/>
-    <xacro:robotis_mini_revolute_joint name="hip_m2_to_hip_m2_plate2" parent_link="hip_m2" child_link="hip_m2_plate2" axis_xyz="0 -1 0" origin_xyz="0.0 0 0.017" origin_rpy="${PI/2.0} 0 ${PI/2.0}" />
+    <xacro:robotis_mini_revolute_joint name="right_hip1" parent_link="hip_m2" child_link="hip_m2_plate2" axis_xyz="0 -1 0" origin_xyz="0.0 0 0.017" origin_rpy="${PI/2.0} 0 ${PI/2.0}" />
   </xacro:macro>
 </robot>
