Commit message: Added friction to all links with a macro

File: robotis_mini_ros/robotis_mini_description/urdf/common.urdf.xacro (robot description, xacro)
@@ -55,4 +55,14 @@
   <property name="MESHVOLUME_XL320"  value="16403.394531" />
   -->
+  <xacro:macro name="friction_properties" params="link_name">
+    <gazebo reference="${link_name}_link">
+      <mu1>10000</mu1>
+      <mu2>10000</mu2>
+      <kp>100.0</kp>
+      <kd>100.0</kd>
+      <minDepth>0.001</minDepth>
+      <maxContacts>100</maxContacts>
+    </gazebo>
+  </xacro:macro>
   <xacro:macro name="robotis_mini_dmfb01" params="name parent xyz rpy">
     <joint name="${name}_joint" type="fixed">
@@ -83,4 +93,5 @@
       </collision>
     </link>
+    <xacro:friction_properties link_name="${name}"/>
   </xacro:macro>
   <xacro:macro name="robotis_mini_dmbb02" params="name parent xyz rpy">
@@ -112,4 +123,5 @@
       </collision>
     </link>
+    <xacro:friction_properties link_name="${name}"/>
   </xacro:macro>
   <xacro:macro name="robotis_mini_dmfb03" params="name parent xyz rpy">
@@ -141,4 +153,5 @@
       </collision>
     </link>
+    <xacro:friction_properties link_name="${name}"/>
   </xacro:macro>
   <xacro:macro name="robotis_mini_dmfb04" params="name parent xyz rpy">
@@ -170,4 +183,5 @@
       </collision>
     </link>
+    <xacro:friction_properties link_name="${name}"/>
   </xacro:macro>
   <xacro:macro name="robotis_mini_dmfb05" params="name parent xyz rpy">
@@ -199,4 +213,5 @@
       </collision>
     </link>
+    <xacro:friction_properties link_name="${name}"/>
   </xacro:macro>
   <xacro:macro name="robotis_mini_dmfb06" params="name parent xyz rpy">
@@ -228,4 +243,5 @@
       </collision>
     </link>
+    <xacro:friction_properties link_name="${name}"/>
   </xacro:macro>
   <xacro:macro name="robotis_mini_dmfb07" params="name parent xyz rpy">
@@ -257,12 +273,5 @@
       </collision>
     </link>
-    <gazebo reference="${name}_link">
-      <mu1>10000</mu1>
-    <mu2>10000</mu2>
-    <kp>10.0</kp>
-    <kd>100.0</kd>
-    <minDepth>0.001</minDepth>
-    <maxContacts>100</maxContacts>
-    </gazebo>
+    <xacro:friction_properties link_name="${name}"/>
   </xacro:macro>
   <xacro:macro name="robotis_mini_dmff01" params="name parent xyz rpy">
@@ -294,4 +303,5 @@
       </collision>
     </link>
+    <xacro:friction_properties link_name="${name}"/>
   </xacro:macro>
   <xacro:macro name="robotis_mini_spu5" params="name parent xyz rpy">
@@ -323,4 +333,5 @@
       </collision>
     </link>
+    <xacro:friction_properties link_name="${name}"/>
   </xacro:macro>
   <xacro:macro name="robotis_mini_spd3b3" params="name parent xyz rpy">
@@ -352,4 +363,5 @@
       </collision>
     </link>
+    <xacro:friction_properties link_name="${name}"/>
   </xacro:macro>
   <xacro:macro name="robotis_mini_spd3b5" params="name parent xyz rpy">
@@ -381,4 +393,5 @@
       </collision>
     </link>
+    <xacro:friction_properties link_name="${name}"/>
   </xacro:macro>
   <xacro:macro name="robotis_mini_spd3b7" params="name parent xyz rpy">
@@ -410,4 +423,5 @@
       </collision>
     </link>
+    <xacro:friction_properties link_name="${name}"/>
   </xacro:macro>
   <xacro:macro name="robotis_mini_spd4b5" params="name parent xyz rpy">
@@ -439,4 +453,5 @@
       </collision>
     </link>
+    <xacro:friction_properties link_name="${name}"/>
   </xacro:macro>
   <xacro:macro name="robotis_mini_spd7v4" params="name parent xyz rpy">
@@ -468,4 +483,5 @@
       </collision>
     </link>
+    <xacro:friction_properties link_name="${name}"/>
   </xacro:macro>
   <xacro:macro name="robotis_mini_spl2b2" params="name parent xyz rpy">
@@ -497,4 +513,5 @@
       </collision>
     </link>
+    <xacro:friction_properties link_name="${name}"/>
   </xacro:macro>
   <xacro:macro name="robotis_mini_spo5" params="name parent xyz rpy">
@@ -526,4 +543,5 @@
       </collision>
     </link>
+    <xacro:friction_properties link_name="${name}"/>
   </xacro:macro>
   <xacro:macro name="robotis_mini_lb040" params="name parent xyz rpy">
@@ -555,4 +573,5 @@
       </collision>
     </link>
+    <xacro:friction_properties link_name="${name}"/>
   </xacro:macro>
   <xacro:macro name="robotis_mini_xl320" params="name">
@@ -579,4 +598,5 @@
       </collision>
     </link>
+    <xacro:friction_properties link_name="${name}"/>
     <gazebo reference="${name}_link">
       <material>Gazebo/DarkGrey</material>
