Commit message: Added virtual camera to the model (cyclop)

File: robotis_mini_ros/robotis_mini_description/urdf/base.urdf.xacro (robot description, xacro)
@@ -6,4 +6,31 @@
   <xacro:macro name="robotis_mini_base" params="name">
     <link name="${name}_link" />
+    <!-- Camera -->
+    <link name="camera_link">
+      <collision>
+        <origin xyz="-0.008 0 0" rpy="0 ${M_PI/2.0 + M_PI/15.0} 0"/>
+        <geometry>
+          <cylinder radius="0.005" length="0.05"/>
+        </geometry>
+      </collision>
+      <visual>
+        <origin xyz="-0.008 0 0" rpy="0 ${M_PI/2.0 + M_PI/15.0} 0"/>
+        <geometry>
+          <cylinder radius="0.005" length="0.05"/>
+        </geometry>
+        <material name="Red"/>
+      </visual>
+      <inertial>
+        <mass value="1e-5" />
+        <origin xyz="-0.008 0 0" rpy="0 ${M_PI/2.0 + M_PI/15.0} 0"/>
+        <inertia ixx="1e-6" ixy="0" ixz="0" iyy="1e-6" iyz="0" izz="1e-6" />
+      </inertial>
+    </link>
+    <joint name="camera_joint" type="fixed">
+      <axis xyz="1 0 0" />
+      <origin xyz="-0.01 0 0.1" rpy="0 0 0"/>
+      <parent link="${name}_link"/>
+      <child link="camera_link"/>
+    </joint>
   </xacro:macro>
 </robot>

File: robotis_mini_ros/robotis_mini_description/urdf/robotis_mini.urdf.xacro (robot description, xacro)
@@ -24,3 +24,43 @@
     </plugin>
   </gazebo>
+    <!-- camera -->
+  <gazebo reference="camera_link">
+    <sensor type="camera" name="camera">
+      <update_rate>30.0</update_rate>
+      <camera name="head">
+        <horizontal_fov>1.3962634</horizontal_fov>
+        <image>
+          <width>640</width>
+          <height>480</height>
+          <format>R8G8B8</format>
+        </image>
+        <clip>
+          <near>0.02</near>
+          <far>300</far>
+        </clip>
+        <noise>
+          <type>gaussian</type>
+          <!-- Noise is sampled independently per pixel on each frame.
+               That pixel's noise value is added to each of its color
+               channels, which at that point lie in the range [0,1]. -->
+          <mean>0.0</mean>
+          <stddev>0.007</stddev>
+        </noise>
+      </camera>
+      <plugin name="camera_controller" filename="libgazebo_ros_camera.so">
+        <alwaysOn>true</alwaysOn>
+        <updateRate>0.0</updateRate>
+        <cameraName>robotis_mini/camera1</cameraName>
+        <imageTopicName>image_raw</imageTopicName>
+        <cameraInfoTopicName>camera_info</cameraInfoTopicName>
+        <frameName>camera_link</frameName>
+        <hackBaseline>0.07</hackBaseline>
+        <distortionK1>0.0</distortionK1>
+        <distortionK2>0.0</distortionK2>
+        <distortionK3>0.0</distortionK3>
+        <distortionT1>0.0</distortionT1>
+        <distortionT2>0.0</distortionT2>
+      </plugin>
+    </sensor>
+  </gazebo>
 </robot>

Commit message: Added camera on the head

File: robotis_mini_ros/robotis_mini_description/urdf/base.urdf.xacro (robot description, xacro)
@@ -11,9 +11,9 @@
         <origin xyz="-0.008 0 0" rpy="0 ${M_PI/2.0 + M_PI/15.0} 0"/>
         <geometry>
-          <cylinder radius="0.005" length="0.05"/>
+          <cylinder radius="0.004" length="0.05"/>
         </geometry>
       </collision>
       <visual>
-        <origin xyz="-0.008 0 0" rpy="0 ${M_PI/2.0 + M_PI/15.0} 0"/>
+        <origin xyz="0 0 -0.025" rpy="0 0 0"/>
         <geometry>
           <cylinder radius="0.005" length="0.05"/>
@@ -23,11 +23,10 @@
       <inertial>
         <mass value="1e-5" />
-        <origin xyz="-0.008 0 0" rpy="0 ${M_PI/2.0 + M_PI/15.0} 0"/>
+        <origin xyz="-0.008 0 0.05" rpy="0 ${M_PI/2.0 + M_PI/15.0} 0"/>
         <inertia ixx="1e-6" ixy="0" ixz="0" iyy="1e-6" iyz="0" izz="1e-6" />
       </inertial>
     </link>
     <joint name="camera_joint" type="fixed">
-      <axis xyz="1 0 0" />
-      <origin xyz="-0.01 0 0.1" rpy="0 0 0"/>
+      <origin xyz="0.0048 0 0.097" rpy="${-M_PI/2.0 - M_PI/20.0} 0 ${-M_PI/2.0}"/>
       <parent link="${name}_link"/>
       <child link="camera_link"/>

Commit message: first with neck

File: robotis_mini_ros/robotis_mini_description/urdf/base.urdf.xacro (robot description, xacro)
@@ -6,30 +6,4 @@
   <xacro:macro name="robotis_mini_base" params="name">
     <link name="${name}_link" />
-    <!-- Camera -->
-    <link name="camera_link">
-      <collision>
-        <origin xyz="-0.008 0 0" rpy="0 ${M_PI/2.0 + M_PI/15.0} 0"/>
-        <geometry>
-          <cylinder radius="0.004" length="0.05"/>
-        </geometry>
-      </collision>
-      <visual>
-        <origin xyz="0 0 -0.025" rpy="0 0 0"/>
-        <geometry>
-          <cylinder radius="0.005" length="0.05"/>
-        </geometry>
-        <material name="Red"/>
-      </visual>
-      <inertial>
-        <mass value="1e-5" />
-        <origin xyz="-0.008 0 0.05" rpy="0 ${M_PI/2.0 + M_PI/15.0} 0"/>
-        <inertia ixx="1e-6" ixy="0" ixz="0" iyy="1e-6" iyz="0" izz="1e-6" />
-      </inertial>
-    </link>
-    <joint name="camera_joint" type="fixed">
-      <origin xyz="0.0048 0 0.097" rpy="${-M_PI/2.0 - M_PI/20.0} 0 ${-M_PI/2.0}"/>
-      <parent link="${name}_link"/>
-      <child link="camera_link"/>
-    </joint>
   </xacro:macro>
 </robot>

File: robotis_mini_ros/robotis_mini_description/urdf/body.urdf.xacro (robot description, xacro)
@@ -13,6 +13,6 @@
     <xacro:robotis_mini_lb040 name="body_chest" parent="body_skeleton_link"
         xyz="0 0.016 -0.004" rpy="0 0 0" />
-    <xacro:robotis_mini_servo_rotating_fake name="neck" parent="body_torso_link"
-        xyz="0 0.036 0.006" rpy="${M_PI/2} 0 0" initial_rotation="0" />
+    <xacro:robotis_mini_servo_rotating name="neck" parent="body_torso_link"
+        xyz="0 0.036 0.006" rpy="${M_PI/2} 0 0" initial_rotation="0" reflect="1"/>
     <xacro:robotis_mini_dmff01 name="body_head" parent="neck_link"
         xyz="0 0 0.003" rpy="${-M_PI/2} 0 0" />

File: robotis_mini_ros/robotis_mini_description/urdf/common.urdf.xacro (robot description, xacro)
@@ -303,4 +303,30 @@
       </collision>
     </link>
+    <!-- Camera  - M_PI/20.0 -->
+    <link name="camera_link">
+      <collision>
+        <origin xyz="-0.008 0 0" rpy="0 ${M_PI/2.0 + M_PI/15.0} 0"/>
+        <geometry>
+          <cylinder radius="0.004" length="0.05"/>
+        </geometry>
+      </collision>
+      <visual>
+        <origin xyz="0 0 -0.025" rpy="0 0 0"/>
+        <geometry>
+          <cylinder radius="0.005" length="0.05"/>
+        </geometry>
+        <material name="Red"/>
+      </visual>
+      <inertial>
+        <mass value="1e-5" />
+        <origin xyz="-0.008 0 0.05" rpy="0 ${M_PI/2.0 + M_PI/15.0} 0"/>
+        <inertia ixx="1e-6" ixy="0" ixz="0" iyy="1e-6" iyz="0" izz="1e-6" />
+      </inertial>
+    </link>
+    <joint name="camera_joint" type="fixed">
+      <origin xyz="0.0 0.022 0.015" rpy="${- M_PI/20.0} 0 ${M_PI}"/>
+      <parent link="${name}_link"/>
+      <child link="camera_link"/>
+    </joint>
     <xacro:friction_properties link_name="${name}"/>
   </xacro:macro>

File: robotis_mini_ros/robotis_mini_description/urdf/servo.urdf.xacro (robot description, xacro)
@@ -29,5 +29,5 @@
     <joint name="${name}_joint" type="revolute">
       <axis xyz="0 0 ${-reflect}" />
-      <limit lower="${-M_PI/2.0}" upper="${M_PI/2.0}" effort="${XL320_MAX_TORQUE}" velocity="${XL320_MAX_VELOCITY}" />
+      <limit lower="${-3*M_PI/4.0}" upper="${3*M_PI/4.0}" effort="${XL320_MAX_TORQUE}" velocity="${XL320_MAX_VELOCITY}" />
       <origin xyz="0 0 0" rpy="0 0 ${initial_rotation}" />
       <parent link="${name}_servo_link"/>
